File: stm32myPill/stm32myPill.kicad_pcb (KiCad board)
At the start: 2 copper layers, 42.4 x 34.8 mm, 32 parts, among them J1 USB_B_Micro, J2 Conn_01x04_Male, J3 Conn_01x04_Male, J4 Conn_01x04_Male, SW1 SW_SPDT, U1 AMS1117-3.3, U2 STM32F103C8T6, Y1 16MHz

Commit message: finished pcb
Parts:
- added G***: LOGO, LOGO, F.Cu at (82.9, 88.0)
- moved R2 11.4 mm to (85.0, 72.9), turned to 90 degrees
- moved R3 1.88 mm to (108.8, 78.1)
- moved C12 1.28 mm to (89.2, 77.7)
- moved C13 1.28 mm to (89.2, 79.9)
- moved Y1 1.28 mm to (86.4, 78.9)
- moved C6 0.67 mm to (101.0, 86.1)
- moved C3 0.44 mm to (95.6, 71.9)
- moved D1 0.27 mm to (115.2, 90.4)
- moved C7 0.22 mm to (104.1, 77.5)
- moved R1 0.12 mm to (115.7, 86.4)
Connections:
- J1 pad 6: unconnected-(J1-Pad6) -> (no net)
Routing:
- net +3V3: track 0.00 -> 158.9 mm, vias 0 -> 4
- net GND: track 0.00 -> 27.5 mm, vias 0 -> 20
- net /BOOT0: track 0.00 -> 22.2 mm
- net /USART1_RX: track 0.00 -> 17.4 mm
- net /SWDIO: track 0.00 -> 17.2 mm
- net /USART1_TX: track 0.00 -> 16.3 mm
- net /USB_D-: track 0.00 -> 13.1 mm
- net /USB_D+: track 0.00 -> 13.1 mm
- net /SWCLK: track 0.00 -> 12.9 mm
- net /I2C2_SCL: track 0.00 -> 12.6 mm
- net /I2C2_SDA: track 0.00 -> 11.1 mm
- net /HSE_IN: track 0.00 -> 9.65 mm
- net /NRST: track 0.00 -> 7.36 mm
- net /HSE_OUT: track 0.00 -> 7.02 mm
- net +3.3VA: track 0.00 -> 6.61 mm
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- added copper zone on F.Cu, net +3V3
- added copper zone on B.Cu, net GND
- added copper zone on F.Cu, net GND
- added copper zone on F.Cu, net VBUS
Other:
- board text added: "-"
- board text added: "BOOT"
- board text added: "CLK"
- board text added: "DIO"
- board text added: "GND"
- board text added: "I2C"
- board text added: "ON"
- board text added: "RX"
- board text added: "STM32 MyPill"
- board text added: "SWD"
- board text added: "TX"
- board text added: "UART"
- board text added: "USB"
- board text added: "V0.1 02/22 Suri Labs"

Commit message: added manafacturing files
Other:
- board text added: "SCL"
- board text added: "SDA"
Changed lines of the file:
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@@
   (gr_line (start 121.412 97.282) (end 78.994 97.282) (layer "Edge.Cuts") (width 0.1))
   (gr_line (start 121.412 62.484) (end 121.412 93.98) (layer "Edge.Cuts") (width 0.1))
+  (gr_text "GND" (at 101.5 92.5) (layer "B.SilkS")
+    (effects (font (size 1 1) (thickness 0.15)) (justify mirror))
+  )
+  (gr_text "SCL\n" (at 95.3 92.5) (layer "B.SilkS")
+    (effects (font (size 1 1) (thickness 0.15)) (justify mirror))
+  )
   (gr_text "TX" (at 95.5 67.6) (layer "B.SilkS")
     (effects (font (size 1 1) (thickness 0.15)) (justify mirror))
@@
     (effects (font (size 1 1) (thickness 0.15)) (justify mirror))
   )
+  (gr_text "SDA" (at 98.4 92.5) (layer "B.SilkS")
+    (effects (font (size 1 1) (thickness 0.15)) (justify mirror))
+  )
